Commit message: copied from multi-mighty branch in mighty repo

File: urdf/dyn_obstacle1.urdf.xacro (robot description, xacro)
@@ -6,4 +6,5 @@
   <xacro:arg name="traj_y" default="cos(t)" />
   <xacro:arg name="traj_z" default="2.0" />
+  <xacro:arg name="size" default="1.0" />
   <!-- Color definitions -->
   <material name="grey">
@@ -19,7 +20,12 @@
       <origin xyz="0 0 0" rpy="0 0 0" />
       <geometry>
-        <mesh filename="$(find dynus)/meshes/obstacles/model4.dae" scale="1.0 1.0 1.0"/>
+        <mesh filename="$(find mighty)/meshes/obstacles/model4.dae" scale="$(arg size) $(arg size) $(arg size)" />
       </geometry>
     </visual>
+    <collision>
+      <geometry>
+        <box size="1.0 1.0 1.0"/>
+      </geometry>
+    </collision>
   </link>
   <!-- Disable gravity for the obstacle -->

File: urdf/quadrotor.urdf.xacro (robot description, xacro)
@@ -7,5 +7,5 @@
     <!-- <xacro:property name="M_PI" value="3.1415926535897931" /> -->
     <!-- Included URDF Files -->
-    <xacro:include filename="$(find dynus)/urdf/quadrotor_base.urdf.xacro" />
+    <xacro:include filename="$(find mighty)/urdf/quadrotor_base.urdf.xacro" />
     <!-- Instantiate quadrotor_base_macro once (has no parameters atm) -->
     <xacro:quadrotor_base_macro />
@@ -14,13 +14,13 @@
     <xacro:include filename="$(find ros2_livox_simulation)/urdf/mid360.xacro" />
     <xacro:mid360 name="$(arg namespace)_livox" namespace="$(arg namespace)" parent="base_link" topic="mid360" >
-      <origin xyz="0 0 0.0" rpy="0 0 0"/>
+      <origin xyz="0 0 0.2" rpy="0 0.3 0"/>
     </xacro:mid360>
     <!-- Forward facing camera (d435)-->
-    <xacro:include filename="$(find dynus)/urdf/_d435.urdf.xacro" />
+    <xacro:include filename="$(find mighty)/urdf/_d435.urdf.xacro" />
     <xacro:sensor_d435 name="$(arg namespace)_d435" topics_ns="$(arg namespace)" range_max_depth="$(arg d435_range_max_depth)" parent="base_link">
       <origin xyz="0.05 0.0 0" rpy="0 0 0"/>
     </xacro:sensor_d435>
     <!-- Forward facing camera (d435i)-->
-    <!-- <xacro:include filename="$(find dynus)/urdf/_d435i.urdf.xacro" />
+    <!-- <xacro:include filename="$(find mighty)/urdf/_d435i.urdf.xacro" />
     <xacro:sensor_d435i name="$(arg namespace)_d435i" topics_ns="$(arg namespace)" parent="base_link">
       <origin xyz="0.2 0.0 0" rpy="0 0 0"/>
@@ -28,15 +28,15 @@
     <!-- Forward facing camera -->
     <!-- TODO: Not sure why but can't put them in namespace  -->
-    <!-- <xacro:include filename="$(find dynus)/urdf/generic_camera.urdf.xacro" />
+    <!-- <xacro:include filename="$(find mighty)/urdf/generic_camera.urdf.xacro" />
     <xacro:generic_camera name="$(arg namespace)_front_cam" parent="base_link" ros_topic="$(arg namespace)" cam_info_topic="$(arg namespace)" update_rate="50" res_x="320" res_y="240" image_format="R8G8B8" hfov="90">
       <origin xyz="0.1 0.0 -0.1" rpy="0 0 0"/>
     </xacro:generic_camera> -->
     <!-- Forward facing camera (t265)-->
-    <!-- <xacro:include filename="$(find dynus)/urdf/_t265.urdf.xacro" />
+    <!-- <xacro:include filename="$(find mighty)/urdf/_t265.urdf.xacro" />
     <xacro:sensor_t265 name="front_cam" topics_ns="$(arg namespace)" parent="base_link">
       <origin xyz="0.1 0.0 0.1" rpy="0 0 0"/>
     </xacro:sensor_t265> -->
     <!-- Sonar height sensor -->
-    <!-- <xacro:include filename="$(find dynus)/urdf/sonar_sensor.urdf.xacro" />
+    <!-- <xacro:include filename="$(find mighty)/urdf/sonar_sensor.urdf.xacro" />
     <xacro:sonar_sensor name="sonar" parent="base_link" >
       <origin xyz="-0.03 -0.03 1.0" rpy="0 ${90*pi/180} 0"/>
