Commit message: rename from mighty to dynus

File: urdf/_d435.urdf.xacro (robot description, xacro)
@@ -8,5 +8,5 @@
 <robot name="sensor_d435" xmlns:xacro="http://ros.org/wiki/xacro">
   <!--File includes-->
-  <xacro:include filename="$(find mighty)/urdf/_d435.gazebo.xacro"/>
+  <xacro:include filename="$(find dynus)/urdf/_d435.gazebo.xacro"/>
   <xacro:macro name="sensor_d435" params="name:=camera topics_ns range_max_depth parent *origin publish_pointcloud:=true">
     <xacro:property name="M_PI" value="3.1415926535897931" />
@@ -48,5 +48,5 @@
         <geometry>
           <!-- <box size="${d435_cam_width} ${d435_cam_height} ${d435_cam_depth}"/> -->
-          <mesh filename="package://mighty/share/dynus/meshes/real_sense/d435.dae" />
+          <mesh filename="package://dynus/share/dynus/meshes/real_sense/d435.dae" />
         </geometry>
         <material name="${name}_aluminum"/>

File: urdf/_d435i.urdf.xacro (robot description, xacro)
@@ -11,5 +11,5 @@
 <robot name="sensor_d435i" xmlns:xacro="http://ros.org/wiki/xacro">
   <!--File includes-->
-  <xacro:include filename="$(find mighty)/urdf/_d435i.gazebo.xacro"/>
+  <xacro:include filename="$(find dynus)/urdf/_d435i.gazebo.xacro"/>
   <xacro:macro name="sensor_d435i" params="parent
                                           name:=camera
@@ -69,5 +69,5 @@
       <origin xyz="${d435i_cam_mount_from_center_offset} ${-d435i_cam_depth_py} 0" rpy="${M_PI/2} 0 ${M_PI/2}"/>
         <geometry>
-          <mesh filename="package://mighty/share/dynus/meshes/real_sense/d435.dae"/>
+          <mesh filename="package://dynus/share/dynus/meshes/real_sense/d435.dae"/>
         </geometry>
         <material name="${name}_aluminum"/>

File: urdf/_t265.urdf.xacro (robot description, xacro)
@@ -12,5 +12,5 @@
 <robot name="sensor_t265" xmlns:xacro="http://ros.org/wiki/xacro">
   <!--File includes-->
-  <xacro:include filename="$(find mighty)/urdf/_t265.gazebo.xacro"/>
+  <xacro:include filename="$(find dynus)/urdf/_t265.gazebo.xacro"/>
     <!-- odom_xyz, odom_rpy params are the transformation from the robot base_link to the camera reference frame (camerea_pose_frame)
   they are needed for the simulation of the camera slam capabilities -->

File: urdf/dyn_obstacle1.urdf.xacro (robot description, xacro)
@@ -20,5 +20,5 @@
       <origin xyz="0 0 0" rpy="0 0 0" />
       <geometry>
-        <mesh filename="$(find mighty)/meshes/obstacles/model4.dae" scale="$(arg size) $(arg size) $(arg size)" />
+        <mesh filename="$(find dynus)/meshes/obstacles/model4.dae" scale="$(arg size) $(arg size) $(arg size)" />
       </geometry>
     </visual>

File: urdf/p3at.urdf.xacro (robot description, xacro)
@@ -18,5 +18,5 @@
   <xacro:arg name="namespace" default="NX01" />
   <xacro:arg name="d435_range_max_depth" default="5.0" />
-  <xacro:include filename="$(find mighty)/urdf/pioneer3at_body.urdf.xacro" />
+  <xacro:include filename="$(find dynus)/urdf/pioneer3at_body.urdf.xacro" />
   <xacro:p3at_gazebo_ext name="$(arg namespace)_red_rover" namespace="$(arg namespace)" />
   <xacro:include filename="$(find ros2_livox_simulation)/urdf/mid360.xacro" />
@@ -24,5 +24,5 @@
     <origin xyz="0 0 1.0" rpy="0 0 0"/>
   </xacro:mid360>
-  <xacro:include filename="$(find mighty)/urdf/_d435.urdf.xacro" />
+  <xacro:include filename="$(find dynus)/urdf/_d435.urdf.xacro" />
   <xacro:sensor_d435 name="$(arg namespace)_d435" topics_ns="$(arg namespace)" range_max_depth="$(arg d435_range_max_depth)" parent="base_link">
     <origin xyz="1.0 0.0 1.0" rpy="0 0 0"/>

File: urdf/p3at_manual.urdf (robot description, URDF)
Before this commit: robot rover, 16 links, 15 joints
Links:
- link chassis: geometry collision mesh filename=$(find dynus)/meshes/chassis.dae; visual mesh filename=$(find dynus)/meshes/chassis.dae
- link laser_link: geometry collision box size=0.01 0.01 0.01; visual mesh filename=$(find dynus)/meshes/hokuyo1.dae
- link p3at_back_left_axle: geometry collision mesh filename=$(find dynus)/meshes/axle.dae; visual mesh filename=$(find dynus)/meshes/axle.dae
- link p3at_back_left_hub: geometry collision mesh filename=$(find dynus)/meshes/left_hubcap.dae; visual mesh filename=$(find dynus)/meshes/left_hubcap.dae
- link p3at_back_left_wheel: geometry collision cylinder length=0.035 radius=0.110; visual mesh filename=$(find dynus)/meshes/left_wheel.dae
- link p3at_back_right_axle: geometry collision mesh filename=$(find dynus)/meshes/axle.dae; visual mesh filename=$(find dynus)/meshes/axle.dae
- link p3at_back_right_hub: geometry collision mesh filename=$(find dynus)/meshes/right_hubcap.dae; visual mesh filename=$(find dynus)/meshes/right_hubcap.dae
- link p3at_back_right_wheel: geometry collision cylinder length=0.035 radius=0.110; visual mesh filename=$(find dynus)/meshes/right_wheel.dae
- link p3at_front_left_axle: geometry collision box size=0 0 0; visual mesh filename=$(find dynus)/meshes/axle.dae
- link p3at_front_left_hub: geometry collision box size=0 0 0; visual mesh filename=$(find dynus)/meshes/left_hubcap.dae
- link p3at_front_left_wheel: geometry collision cylinder length=0.035 radius=0.110; visual mesh filename=$(find dynus)/meshes/left_wheel.dae
- link p3at_front_right_axle: geometry collision box size=0 0 0; visual mesh filename=$(find dynus)/meshes/axle.dae
- link p3at_front_right_hub: geometry collision box size=0 0 0; visual mesh filename=$(find dynus)/meshes/right_hubcap.dae
- link p3at_front_right_wheel: geometry collision cylinder length=0.035 radius=0.110; visual mesh filename=$(find dynus)/meshes/right_wheel.dae
- link top_plate: geometry collision box size=0 0 0; visual mesh filename=$(find dynus)/meshes/top.dae

File: urdf/pioneer3at_body.urdf.xacro (robot description, xacro)
@@ -24,5 +24,5 @@
 			<origin xyz="0 0 0.177" rpy="0 0 0"/>
 			<geometry name="pioneer_geom">
-				<mesh filename="$(find mighty)/meshes/p3at_meshes/chassis.stl"/>
+				<mesh filename="$(find dynus)/meshes/p3at_meshes/chassis.stl"/>
 			</geometry>
 			<material name="ChassisRed">
@@ -33,5 +33,5 @@
 			<origin xyz="0 0 0.177" rpy="0 0 0"/>
 				<geometry>
-					<mesh filename="$(find mighty)/meshes/p3at_meshes/chassis.stl"/>
+					<mesh filename="$(find dynus)/meshes/p3at_meshes/chassis.stl"/>
 				</geometry>
 		</collision>
@@ -52,5 +52,5 @@
 			<origin xyz="0 0 0" rpy="0 0 0"/>
 			<geometry name="pioneer_geom">
-				<mesh filename="$(find mighty)/meshes/p3at_meshes/top.stl"/>
+				<mesh filename="$(find dynus)/meshes/p3at_meshes/top.stl"/>
 			</geometry>
 			<material name="TopBlack">
@@ -78,5 +78,5 @@
 			<origin xyz="0 0 0" rpy="0 0 0"/>
 			<geometry name="pioneer_geom">
-				<mesh filename="$(find mighty)/meshes/p3at_meshes/front_sonar.stl"/>
+				<mesh filename="$(find dynus)/meshes/p3at_meshes/front_sonar.stl"/>
 			</geometry>
 			<material name="SonarYellow">
@@ -103,5 +103,5 @@
 			<origin xyz="0 0 0" rpy="0 0 0"/>
 			<geometry name="pioneer_geom">
-				<mesh filename="$(find mighty)/meshes/p3at_meshes/back_sonar.stl"/>
+				<mesh filename="$(find dynus)/meshes/p3at_meshes/back_sonar.stl"/>
 			</geometry>
 			<material name="SonarYellow">
@@ -130,5 +130,5 @@
 		<origin xyz="0 0 0" rpy="0 0 0"/>
 		<geometry name="pioneer_geom">
-			<mesh filename="$(find mighty)/meshes/p3at_meshes/axle.stl"/>
+			<mesh filename="$(find dynus)/meshes/p3at_meshes/axle.stl"/>
 		</geometry>
 		<material name="AxleGrey">
@@ -155,5 +155,5 @@
 		<origin xyz="0 0 0" rpy="0 0 0"/>
 		<geometry name="pioneer_geom">
-			<mesh filename="$(find mighty)/meshes/p3at_meshes/${side}_hubcap.stl"/>
+			<mesh filename="$(find dynus)/meshes/p3at_meshes/${side}_hubcap.stl"/>
 		</geometry>
 		<material name="HubcapYellow">
@@ -180,5 +180,5 @@
 		<origin xyz="0 0 0" rpy="0 0 0"/>
 		<geometry name="pioneer_geom">
-			<mesh filename="$(find mighty)/meshes/p3at_meshes/wheel.stl"/>
+			<mesh filename="$(find dynus)/meshes/p3at_meshes/wheel.stl"/>
 		</geometry>
 		<material name="WheelBlack">
@@ -189,5 +189,5 @@
 		<origin xyz="0 0 0" rpy="${-3.1415927/2} 0 0"/>
 		<geometry>
-	    <!--mesh filename="$(find mighty)/meshes/p3at_meshes/wheel.stl"/-->
+	    <!--mesh filename="$(find dynus)/meshes/p3at_meshes/wheel.stl"/-->
 	    <cylinder radius="0.111" length="0.075"/>
 		</geometry>
@@ -217,5 +217,5 @@
 		<origin xyz="0 0 0" rpy="0 0 0"/>
 		<geometry name="pioneer_geom">
-			<mesh filename="$(find mighty)/meshes/p3at_meshes/axle.stl"/>
+			<mesh filename="$(find dynus)/meshes/p3at_meshes/axle.stl"/>
 		</geometry>
 		<material name="AxleGrey">
@@ -226,5 +226,5 @@
 		<origin xyz="0 0 0" rpy="0 0 0"/>
 		<geometry>
-			<mesh filename="$(find mighty)/meshes/p3at_meshes/axle.stl"/>
+			<mesh filename="$(find dynus)/meshes/p3at_meshes/axle.stl"/>
 		</geometry>
 	</collision>
@@ -248,5 +248,5 @@
 		<origin xyz="0 0 0" rpy="0 0 0"/>
 		<geometry name="pioneer_geom">
-			<mesh filename="$(find mighty)/meshes/p3at_meshes/${side}_hubcap.stl"/>
+			<mesh filename="$(find dynus)/meshes/p3at_meshes/${side}_hubcap.stl"/>
 		</geometry>
 		<material name="HubcapYellow"/>
@@ -255,5 +255,5 @@
 		<origin xyz="0 0 0" rpy="0 0 0"/>
 		<geometry>
-			<mesh filename="$(find mighty)/meshes/p3at_meshes/${side}_hubcap.stl"/>
+			<mesh filename="$(find dynus)/meshes/p3at_meshes/${side}_hubcap.stl"/>
 		</geometry>
 	</collision>
@@ -278,5 +278,5 @@
 		<origin xyz="0 0 0" rpy="0 0 0"/>
 		<geometry name="pioneer_geom">
-			<mesh filename="$(find mighty)/meshes/p3at_meshes/wheel.stl"/>
+			<mesh filename="$(find dynus)/meshes/p3at_meshes/wheel.stl"/>
 		</geometry>
 		<material name="WheelBlack"/>
@@ -285,5 +285,5 @@
 		<origin xyz="0 0 0" rpy="${-3.1415927/2} 0 0"/>
 		<geometry>
-	    <!--mesh filename="$(find mighty)/meshes/p3at_meshes/wheel.stl"/-->
+	    <!--mesh filename="$(find dynus)/meshes/p3at_meshes/wheel.stl"/-->
 	    <cylinder radius="0.111" length="0.075"/>
 		</geometry>

File: urdf/quadrotor.urdf.xacro (robot description, xacro)
@@ -7,5 +7,5 @@
     <!-- <xacro:property name="M_PI" value="3.1415926535897931" /> -->
     <!-- Included URDF Files -->
-    <xacro:include filename="$(find mighty)/urdf/quadrotor_base.urdf.xacro" />
+    <xacro:include filename="$(find dynus)/urdf/quadrotor_base.urdf.xacro" />
     <!-- Instantiate quadrotor_base_macro once (has no parameters atm) -->
     <xacro:quadrotor_base_macro />
@@ -17,10 +17,10 @@
     </xacro:mid360>
     <!-- Forward facing camera (d435)-->
-    <xacro:include filename="$(find mighty)/urdf/_d435.urdf.xacro" />
+    <xacro:include filename="$(find dynus)/urdf/_d435.urdf.xacro" />
     <xacro:sensor_d435 name="$(arg namespace)_d435" topics_ns="$(arg namespace)" range_max_depth="$(arg d435_range_max_depth)" parent="base_link">
       <origin xyz="0.05 0.0 0" rpy="0 0 0"/>
     </xacro:sensor_d435>
     <!-- Forward facing camera (d435i)-->
-    <!-- <xacro:include filename="$(find mighty)/urdf/_d435i.urdf.xacro" />
+    <!-- <xacro:include filename="$(find dynus)/urdf/_d435i.urdf.xacro" />
     <xacro:sensor_d435i name="$(arg namespace)_d435i" topics_ns="$(arg namespace)" parent="base_link">
       <origin xyz="0.2 0.0 0" rpy="0 0 0"/>
@@ -28,15 +28,15 @@
     <!-- Forward facing camera -->
     <!-- TODO: Not sure why but can't put them in namespace  -->
-    <!-- <xacro:include filename="$(find mighty)/urdf/generic_camera.urdf.xacro" />
+    <!-- <xacro:include filename="$(find dynus)/urdf/generic_camera.urdf.xacro" />
     <xacro:generic_camera name="$(arg namespace)_front_cam" parent="base_link" ros_topic="$(arg namespace)" cam_info_topic="$(arg namespace)" update_rate="50" res_x="320" res_y="240" image_format="R8G8B8" hfov="90">
       <origin xyz="0.1 0.0 -0.1" rpy="0 0 0"/>
     </xacro:generic_camera> -->
     <!-- Forward facing camera (t265)-->
-    <!-- <xacro:include filename="$(find mighty)/urdf/_t265.urdf.xacro" />
+    <!-- <xacro:include filename="$(find dynus)/urdf/_t265.urdf.xacro" />
     <xacro:sensor_t265 name="front_cam" topics_ns="$(arg namespace)" parent="base_link">
       <origin xyz="0.1 0.0 0.1" rpy="0 0 0"/>
     </xacro:sensor_t265> -->
     <!-- Sonar height sensor -->
-    <!-- <xacro:include filename="$(find mighty)/urdf/sonar_sensor.urdf.xacro" />
+    <!-- <xacro:include filename="$(find dynus)/urdf/sonar_sensor.urdf.xacro" />
     <xacro:sonar_sensor name="sonar" parent="base_link" >
       <origin xyz="-0.03 -0.03 1.0" rpy="0 ${90*pi/180} 0"/>

File: urdf/quadrotor_base.urdf.xacro (robot description, xacro)
@@ -14,5 +14,5 @@
         <origin xyz="0 0 0" rpy="0 0 0" />
         <geometry>
-          <mesh filename="$(find mighty)/meshes/quadrotor/quadrotor_base_2.dae" scale="0.5 0.5 0.5"/>
+          <mesh filename="$(find dynus)/meshes/quadrotor/quadrotor_base_2.dae" scale="0.5 0.5 0.5"/>
         </geometry>
       </visual>
@@ -20,5 +20,5 @@
         <origin xyz="0 0 0" rpy="0 0 ${45*pi/180}" />
         <geometry>
-          <mesh filename="$(find mighty)/meshes/quadrotor/quadrotor_base_2.stl"/>
+          <mesh filename="$(find dynus)/meshes/quadrotor/quadrotor_base_2.stl"/>
         </geometry>
       </collision> -->

File: urdf/sonar_sensor.urdf.xacro (robot description, xacro)
@@ -17,5 +17,5 @@
         <geometry>
           <!--<box size="0.01 0.01 0.01" /> -->
-          <mesh filename="package://mighty/share/dynus/meshes/sonar_sensor/max_sonar_ez4.dae"/>
+          <mesh filename="package://dynus/share/dynus/meshes/sonar_sensor/max_sonar_ez4.dae"/>
         </geometry>
       </visual>
